Commit message: vs update

File: src/ROBOTIS_OP3_src/ROBOTIS-OP3-Common/op3_description/urdf/robotis_op3.gazebo.xacro (robot description, xacro)
@@ -4,5 +4,5 @@
     <plugin name="gazebo_ros_control" filename="libgazebo_ros_control.so">
       <robotNamespace>/robotis_op3</robotNamespace>
-      <updateRate>30</updateRate>
+      <updateRate>50</updateRate>
     </plugin>
   </gazebo>

File: src/ROBOTIS_OP3_src/ROBOTIS-OP3-Common/op3_description/urdf/robotis_op3.inertia.xacro (robot description, xacro)
@@ -158,7 +158,7 @@
     <origin xyz="0.00233 0.00000 0.00823" />
     <mass value="0.01176"/>
-    <inertia ixx="0.0001" ixy="0.0" ixz="-0.000"
-             iyy="0.0001" iyz="0.0"
-             izz="0.0001" />
+    <inertia ixx="0.001" ixy="0.0" ixz="-0.001"
+             iyy="0.001" iyz="0.0"
+             izz="0.001" />
   </xacro:macro>
   <!-- head pitch joint -->
@@ -166,5 +166,5 @@
     <origin xyz="0.00230 -0.01863 0.02770" />
     <mass value="0.13631"/>
-    <inertia ixx="0.001" ixy="0.000" ixz="-0.000"
+    <inertia ixx="0.001" ixy="0.000" ixz="-0.001"
              iyy="0.001" iyz="0.000"
              izz="0.001" />

File: src/ROBOTIS_OP3_src/ROBOTIS-OP3-Common/op3_description/urdf/robotis_op3.structure.head.xacro (robot description, xacro)
@@ -10,6 +10,6 @@
     <origin xyz="0.1 0.0 0.003" rpy="0 0 0" />
     <axis xyz="0 0 1" />
-    <limit effort="1000" velocity="100" lower="${-pi*2/3}" upper="${pi*2/3}" />
-    <dynamics damping="0.1" friction="0.0" />
+    <limit effort="1000" velocity="100" lower="${-pi*75/180}" upper="${pi*75/180}" />
+    <dynamics damping="0.1" friction="0.1" />
   </joint>
   <xacro:insert_transmission name="head_pan" />
@@ -32,6 +32,6 @@
     <origin xyz="0.010 0.019 0.0285" rpy="0 0 0" />
     <axis xyz="0 -1 0" />
-    <limit effort="1000" velocity="100" lower="${-pi*0.5}" upper="${pi*0.5}" />
-    <dynamics damping="0.1" friction="0.0" />
+    <limit effort="1000" velocity="100" lower="${-pi*15/180}" upper="${pi*35/180}" />
+    <dynamics damping="0.1" friction="0.1" />
   </joint>
   <xacro:insert_transmission name="head_tilt" />
