Commit message: update from home

File: src/ROBOTIS_OP3_src/ROBOTIS-OP3-Common/op3_description/urdf/robotis_op3.inertia.xacro (robot description, xacro)
@@ -158,7 +158,7 @@
     <origin xyz="0.00233 0.00000 0.00823" />
     <mass value="0.01176"/>
-    <inertia ixx="0.001" ixy="0.0" ixz="-0.001"
-             iyy="0.001" iyz="0.0"
-             izz="0.001" />
+    <inertia ixx="0.00001" ixy="0.0" ixz="-0.00001"
+             iyy="0.00001" iyz="0.0"
+             izz="0.00001" />
   </xacro:macro>
   <!-- head pitch joint -->
@@ -166,7 +166,7 @@
     <origin xyz="0.00230 -0.01863 0.02770" />
     <mass value="0.13631"/>
-    <inertia ixx="0.001" ixy="0.000" ixz="-0.001"
-             iyy="0.001" iyz="0.000"
-             izz="0.001" />
+    <inertia ixx="0.00001" ixy="0.000" ixz="-0.00001"
+             iyy="0.00001" iyz="0.000"
+             izz="0.00001" />
   </xacro:macro>
 </robot>

File: src/ROBOTIS_OP3_src/ROBOTIS-OP3-Common/op3_description/urdf/robotis_op3.structure.head.xacro (robot description, xacro)
@@ -8,5 +8,5 @@
     <parent link="${parent}"/>
     <child link="head_pan_link"/>
-    <origin xyz="0.1 0.0 0.003" rpy="0 0 0" />
+    <origin xyz="0. 0.0 0.003" rpy="0 0 0" />
     <axis xyz="0 0 1" />
     <limit effort="1000" velocity="100" lower="${-pi*75/180}" upper="${pi*75/180}" />

File: src/turtlebot_src/kobuki_description/urdf/kobuki.urdf.xacro (robot description, xacro)
@@ -9,4 +9,5 @@
   <xacro:include filename="$(find kobuki_description)/urdf/common_properties.urdf.xacro"/>
   <xacro:include filename="$(find kobuki_description)/urdf/kobuki_gazebo.urdf.xacro"/>
+  <xacro:include filename="$(find ros_controllers_redefined)/urdf/wheel_transmission.xacro"/>
   <xacro:property name="M_PI" value="3.1415926535897931" />
   <!-- Kobuki -->
@@ -62,5 +63,7 @@
       <origin xyz="0.00 ${0.23/2} 0.0250" rpy="${-M_PI/2} 0 0"/>
       <axis xyz="0 0 1"/>
-    </joint>
+      <!-- <limit effort="6.0" velocity="${1.0 / 0.035}"/> -->
+    </joint>
+    <!-- <xacro:wheel_transmission side="left"/> -->
     <link name="wheel_left_link">
       <visual>
@@ -89,5 +92,7 @@
       <origin xyz="0.00 -${0.23/2} 0.0250" rpy="${-M_PI/2} 0 0"/>
       <axis xyz="0 0 1"/>
-    </joint>
+      <!-- <limit effort="6.0" velocity="${1.0 / 0.035}"/> -->
+    </joint>
+    <!-- <xacro:wheel_transmission side="right"/> -->
     <link name="wheel_right_link">
       <visual>

File: src/turtlebot_src/kobuki_description/urdf/kobuki_gazebo.urdf.xacro (robot description, xacro)
@@ -3,18 +3,22 @@
   <xacro:macro name="kobuki_sim">
 	  <gazebo reference="wheel_left_link">
-	    <mu1>1.0</mu1>
-	    <mu2>1.0</mu2>
-	    <kp>1000000.0</kp>
-	    <kd>100.0</kd>
-	    <minDepth>0.001</minDepth>
+      <kp>1000000.0</kp>
+      <kd>1000.0</kd>
+      <mu1>1.0</mu1>
+      <mu2>0.1</mu2> <!-- Frictionless wheels 0.0-->
+	    <minDepth>0.00</minDepth>
 	    <maxVel>1.0</maxVel>
+      <implicitSpringDamper>1</implicitSpringDamper>
+      <fdir1>1 0 0</fdir1>
 	  </gazebo>
 	  <gazebo reference="wheel_right_link">
-	    <mu1>1.0</mu1>
-	    <mu2>1.0</mu2>
-	    <kp>1000000.0</kp>
-	    <kd>100.0</kd>
-	    <minDepth>0.001</minDepth>
+      <kp>1000000.0</kp>
+      <kd>1000.0</kd>
+      <mu1>1.0</mu1>
+      <mu2>0.1</mu2> <!-- Frictionless wheels 0.0-->
+	    <minDepth>0.00</minDepth>
 	    <maxVel>1.0</maxVel>
+      <implicitSpringDamper>1</implicitSpringDamper>
+      <fdir1>1 0 0</fdir1>
 	  </gazebo>
 	  <gazebo reference="caster_front_link">
@@ -160,4 +164,9 @@
       </sensor>
 	  </gazebo>
+    <!-- <gazebo>
+      <plugin name="gazebo_ros_control" filename="libgazebo_ros_control.so">
+        <updateRate>50</updateRate>
+      </plugin>
+    </gazebo> -->
 	  <gazebo>
 	    <plugin name="kobuki_controller" filename="libgazebo_ros_kobuki.so">
