Commit message: Pan + Mobile Base Control

File: src/ROBOTIS_OP3_src/ROBOTIS-OP3-Common/op3_description/urdf/robotis_op3.structure.head.xacro (robot description, xacro)
@@ -8,5 +8,5 @@
     <parent link="${parent}"/>
     <child link="head_pan_link"/>
-    <origin xyz="0.0 0.0 0.003" rpy="0 0 0" />
+    <origin xyz="0.1 0.0 0.003" rpy="0 0 0" />
     <axis xyz="0 0 1" />
     <limit effort="1000" velocity="100" lower="${-pi*2/3}" upper="${pi*2/3}" />

Commit message: Kinematics model

File: src/ROBOTIS_OP3_src/ROBOTIS-OP3-Common/op3_description/urdf/robotis_op3.structure.head.xacro (robot description, xacro)
@@ -11,5 +11,5 @@
     <axis xyz="0 0 1" />
     <limit effort="1000" velocity="100" lower="${-pi*75/180}" upper="${pi*75/180}" />
-    <dynamics damping="0.1" friction="0.1" />
+    <dynamics damping="0.1" friction="0.15" />
   </joint>
   <xacro:insert_transmission name="head_pan" />
@@ -33,5 +33,5 @@
     <axis xyz="0 -1 0" />
     <limit effort="1000" velocity="100" lower="${-pi*15/180}" upper="${pi*35/180}" />
-    <dynamics damping="0.1" friction="0.1" />
+    <dynamics damping="0.1" friction="0.15" />
   </joint>
   <xacro:insert_transmission name="head_tilt" />

Commit message: new turtlebot2 base

File: src/ROBOTIS_OP3_src/ROBOTIS-OP3-Common/op3_description/urdf/robotis_op3.structure.head.xacro (robot description, xacro)
@@ -10,5 +10,5 @@
     <origin xyz="0. 0.0 0.003" rpy="0 0 0" />
     <axis xyz="0 0 1" />
-    <limit effort="1000" velocity="100" lower="${-pi*75/180}" upper="${pi*75/180}" />
+    <limit effort="4" velocity="3" lower="${-pi*75/180}" upper="${pi*75/180}" />
     <dynamics damping="0.1" friction="0.15" />
   </joint>
@@ -32,5 +32,5 @@
     <origin xyz="0.010 0.019 0.0285" rpy="0 0 0" />
     <axis xyz="0 -1 0" />
-    <limit effort="1000" velocity="100" lower="${-pi*15/180}" upper="${pi*35/180}" />
+    <limit effort="4" velocity="3" lower="${-pi*15/180}" upper="${pi*35/180}" />
     <dynamics damping="0.1" friction="0.15" />
   </joint>
