Commit message: ARI Head on Turtlebot2

File: src/turtlebot2_src/src/kobuki_description/urdf/kobuki_gazebo.urdf.xacro (robot description, xacro)
@@ -176,4 +176,24 @@
         <imu_name>imu</imu_name>
 	    </plugin>
+      <plugin filename="libgazebo_ros_control.so" name="gazebo_ros_control">
+        <ns></ns>
+        <!-- <robotSimType>pal_hardware_gazebo/PalHardwareGazebo</robotSimType> -->
+        <!-- <xacro:if value="${is_multiple}">
+            <robotNamespace>/${nsp}</robotNamespace>
+        </xacro:if>
+        <xacro:unless value="${is_multiple}">
+            <robotNamespace></robotNamespace>
+        </xacro:unless> -->
+        <!-- <controlPeriod>0.001</controlPeriod> -->
+      </plugin>
+      <plugin filename="libgazebo_ros_p3d.so" name="gazebo_ros_p3d">
+      <bodyName>base_footprint</bodyName>
+      <topicName>ground_truth_odom</topicName>
+      <alwaysOn>true</alwaysOn>
+      <updateRate>100.0</updateRate>
+      <!-- <xacro:if value="${is_multiple}">
+          <robotNamespace>/${nsp}</robotNamespace>
+      </xacro:if> -->
+    </plugin>
 	  </gazebo>
   </xacro:macro>

File: src/turtlebot2_src/src/turtlebot/turtlebot_description/urdf/stacks/hexagons_extended.urdf.xacro (robot description, xacro)
@@ -5,9 +5,12 @@
 <robot name="stack_hexagons" xmlns:xacro="http://ros.org/wiki/xacro">
   <xacro:include filename="$(find turtlebot_description)/urdf/common_properties.urdf.xacro"/>
-  <xacro:include filename="$(find op3_description)/urdf/robotis_op3.visuals.xacro" />
-  <xacro:include filename="$(find op3_description)/urdf/robotis_op3.inertia.xacro" />
-  <xacro:include filename="$(find op3_description)/urdf/robotis_op3.structure.head.xacro" />
-  <xacro:include filename="$(find op3_description)/urdf/robotis_op3.gazebo.xacro" />
-  <xacro:include filename="$(find op3_description)/urdf/robotis_op3.transmissions.xacro" />
+  <!-- <xacro:include filename="$(find op3_description)/urdf/robotis_op3.visuals.xacro" /> -->
+  <!-- <xacro:include filename="$(find op3_description)/urdf/robotis_op3.inertia.xacro" /> -->
+  <!-- <xacro:include filename="$(find op3_description)/urdf/robotis_op3.structure.head.xacro" /> -->
+  <!-- <xacro:include filename="$(find op3_description)/urdf/robotis_op3.gazebo.xacro" /> -->
+  <!-- <xacro:include filename="$(find op3_description)/urdf/robotis_op3.transmissions.xacro" /> -->
+  <xacro:include filename="$(find ari_description)/urdf/head/head.urdf.xacro" />
+  <!-- Generic simulator_gazebo plugins -->
+  <!-- <xacro:include filename="$(find ari_description)/gazebo/gazebo.urdf.xacro" /> -->
   <!-- Xacro properties -->
   <xacro:property name="M_SCALE" value="0.001"/>
@@ -286,5 +289,7 @@
       </inertial>
     </link>
-    <xacro:robotis_op3_head parent="plate_top_3rd_link" />
+    <!-- <xacro:robotis_op3_head parent="plate_top_3rd_link" /> -->
+    <xacro:property name="head_link_name"          value="head_2_link"/>
+    <xacro:head name="head" parent="${parent}"/>
   </xacro:macro>
 </robot>
