Commit message: publish head joints through tf

File: src/head_src/src/ari_head/ari_description/urdf/head/head.urdf.xacro (robot description, xacro)
@@ -36,5 +36,5 @@
       </inertial>
       <visual>
-        <origin xyz="0 0 0.10" rpy="0 0 0"/>
+        <origin xyz="0 0 0" rpy="0 0 0"/>
         <geometry>
           <cylinder radius="0.055" length="0.15"/>
@@ -55,5 +55,5 @@
       <parent link="${parent}"/>
       <child link="${name}_link"/>
-      <origin xyz="-0.0 0 0.8"  rpy="0 0 0" />
+      <origin xyz="-0.0 0 .88"  rpy="0 0 0" />
       <axis xyz="0 0 1" />
       <limit lower="${head_1_lower_limit * deg_to_rad}" upper="${head_1_upper_limit * deg_to_rad}" effort="3.4" velocity="${head_max_vel}" />
@@ -106,5 +106,5 @@
       <parent link="${parent}"/>
       <child link="${name}_link"/>
-      <origin xyz="0.0425000000000001 0 0.093"  rpy="${90.0 * deg_to_rad} 0 0" />
+      <origin xyz="0.0425000000000001 0 0.0"  rpy="${90.0 * deg_to_rad} 0 0" />
       <axis xyz="0 0 -1" />
       <limit lower="${head_2_lower_limit * deg_to_rad}" upper="${head_2_upper_limit * deg_to_rad}" effort="3.26" velocity="${head_max_vel}" />
@@ -124,41 +124,41 @@
   <!--************************-->
   <xacro:macro name="head_front_camera" params="name parent">
-  <link name="${name}_link">
-    <inertial>
-      <origin xyz="-0.00619317919404934 -4.45435622691566E-05 -8.22112600169511E-05" rpy="0 0 0"/>
-      <mass value="0.00115745344894968"/>
-      <inertia ixx="6.76913771029748E-08" ixy="2.52492243040059E-13" ixz="-3.60412180500293E-11"
-               iyy="2.88827920072855E-08" iyz="-1.65336506314803E-13"
-               izz="3.97290092554434E-08"/>
-    </inertial>
-    <!-- <visual>
-      <origin rpy="0 0 0" xyz="0 0 0" />
-      <geometry>
-        <mesh filename="package://ari_description/meshes/sensors/${name}.stl" scale="1 1 1"/>
-      </geometry>
-      <material name="DarkGrey"/>
-    </visual> -->
-    <!-- <collision>
-      <origin rpy="0 0 0" xyz="0 0 0" />
-      <geometry>
-        <mesh filename="package://ari_description/meshes/sensors/${name}.stl" scale="1 1 1"/>
-      </geometry>
-    </collision> -->
-  </link>
-  <joint name="${name}_joint" type="fixed">
-    <origin xyz="0.0633629998680001 0.181996035631448 0" rpy="${-90 * deg_to_rad} 0 0" />
-    <parent link="${parent}" />
-    <child link="${name}_link" />
-    <axis xyz="0 0 0" />
-  </joint>
-  <joint name="${name}_optical_joint" type="fixed">
-    <origin xyz="0.0 0.0 0.0" rpy="${-90 * deg_to_rad} 0 ${-90 * deg_to_rad}" />
-    <parent link="${name}_link" />
-    <child link="${name}_optical_frame" />
-    <axis xyz="0 0 0" />
-  </joint>
-  <link name="${name}_optical_frame"/>
-  <!-- Gazebo plugin -->
-  <xacro:rpi_camera_gazebo name="${name}" topic="${name}" frame="${name}_optical_frame"/>
+    <link name="${name}_link">
+      <inertial>
+        <origin xyz="-0.00619317919404934 -4.45435622691566E-05 -8.22112600169511E-05" rpy="0 0 0"/>
+        <mass value="0.00115745344894968"/>
+        <inertia ixx="6.76913771029748E-08" ixy="2.52492243040059E-13" ixz="-3.60412180500293E-11"
+                 iyy="2.88827920072855E-08" iyz="-1.65336506314803E-13"
+                 izz="3.97290092554434E-08"/>
+      </inertial>
+      <!-- <visual>
+        <origin rpy="0 0 0" xyz="0 0 0" />
+        <geometry>
+          <mesh filename="package://ari_description/meshes/sensors/${name}.stl" scale="1 1 1"/>
+        </geometry>
+        <material name="DarkGrey"/>
+      </visual> -->
+      <!-- <collision>
+        <origin rpy="0 0 0" xyz="0 0 0" />
+        <geometry>
+          <mesh filename="package://ari_description/meshes/sensors/${name}.stl" scale="1 1 1"/>
+        </geometry>
+      </collision> -->
+    </link>
+    <joint name="${name}_joint" type="fixed">
+      <origin xyz="0.0633629998680001 0.181996035631448 0" rpy="${-90 * deg_to_rad} 0 0" />
+      <parent link="${parent}" />
+      <child link="${name}_link" />
+      <axis xyz="0 0 0" />
+    </joint>
+    <joint name="${name}_optical_joint" type="fixed">
+      <origin xyz="0.0 0.0 0.0" rpy="${-90 * deg_to_rad} 0 ${-90 * deg_to_rad}" />
+      <parent link="${name}_link" />
+      <child link="${name}_optical_frame" />
+      <axis xyz="0 0 0" />
+    </joint>
+    <link name="${name}_optical_frame"/>
+    <!-- Gazebo plugin -->
+    <xacro:rpi_camera_gazebo name="${name}" topic="${name}" frame="${name}_optical_frame"/>
   </xacro:macro>
   <xacro:macro name="head" params="name parent">

File: src/turtlebot2_src/src/turtlebot/turtlebot_description/urdf/stacks/hexagons_extended.urdf.xacro (robot description, xacro)
@@ -290,5 +290,5 @@
     </link>
     <!-- <xacro:robotis_op3_head parent="plate_top_3rd_link" /> -->
-    <xacro:property name="head_link_name"          value="head_2_link"/>
+    <!-- <xacro:property name="head_link_name"          value="head_2_link"/> -->
     <xacro:head name="head" parent="${parent}"/>
   </xacro:macro>
